File: customboard/droneboard/droneboard.kicad_sch (KiCad schematic)
At the start: 49 parts, among them J1 Conn_01x04, J3 Conn_01x05_Pin, J4 Conn_01x02_Pin, J7 Conn_01x04_Odd_Even, SW1 SW_Push, SW2 SW_Push, U1 STM32F411CEUx, U3 L78M05CDT, U4 ICM-42688-P, U5 LDK130M33R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

Commit message: stm32f7 initial work
Parts:
- removed J7: Conn_01x04_Odd_Even, Connector_PinHeader_2.54mm:PinHeader_1x04_P2.54mm_Vertical, symbol Connector_Generic:Conn_01x04
- removed U1: STM32F411CEUx, Package_DFN_QFN:QFN-48-1EP_7x7mm_P0.5mm_EP5.6x5.6mm, symbol MCU_ST_STM32F4:STM32F411CEUx
- added C8: 100n, Capacitor_SMD:C_0402_1005Metric, symbol Device:C
- added J2: USB_B_Micro, Connector_USB:USB_Micro-B_Molex_47346-0001, symbol Connector:USB_B_Micro
- added U2: STM32F722RETx, Package_QFP:LQFP-64_10x10mm_P0.5mm, symbol MCU_ST_STM32F7:STM32F722RETx
- J1: footprint Connector_PinHeader_2.54mm:PinHeader_1x04_P2.54mm_Vertical -> Connector_PinHeader_1.27mm:PinHeader_1x04_P1.27mm_Vertical
- J3: footprint Connector_JST:JST_XH_B5B-XH-A_1x05_P2.50mm_Vertical -> Connector_PinHeader_1.27mm:PinHeader_1x05_P1.27mm_Vertical
Connections:
- net BOOT: now also U2.60 (BOOT0)
- net GND: now also C8.2, J2.5 (GND), J2.6 (Shield), U2.12 (VSSA), U2.18 (VSS), U2.31 (VSS), U2.47 (VSS), U2.63 (VSS)
- net RESET1: now also U2.7 (NRST)
- net VMCU: now also C8.1, U2.1 (VBAT), U2.13 (VDDA), U2.19 (VDD), U2.32 (VDD), U2.48 (VDD), U2.64 (VDD)
- net at C15.1: now also U2.30 (VCAP_1)
- net at Y2.1: now also U2.5 (PH0)
- net at Y2.3: now also U2.6 (PH1)
- new net USB_DM: J2.2 (D-), U2.44 (PA11)
- new net USB_DP: J2.3 (D+), U2.45 (PA12)
- no-connect marks 18 -> 2
