File: customboard/droneboard/droneboard.kicad_sch (KiCad schematic)
At the start: 49 parts, among them J1 Conn_01x04, J3 Conn_01x05_Pin, J4 Conn_01x02_Pin, J7 Conn_01x04_Odd_Even, SW1 SW_Push, SW2 SW_Push, U1 STM32F411CEUx, U3 L78M05CDT, U4 ICM-42688-P, U5 LDK130M33R, U6 LDK130M33R, Y2 CSTNE20M0V53Z000R0

Commit message: usb implementation start
Parts:
- removed J7: Conn_01x04_Odd_Even, Connector_PinHeader_2.54mm:PinHeader_1x04_P2.54mm_Vertical, symbol Connector_Generic:Conn_01x04
- added J2: USB_B_Micro, Connector_USB:USB_Micro-B_Molex_47346-0001, symbol Connector:USB_B_Micro
Connections:
- net SWCLK is gone; now on net BLUE: U1.37 (PA14)
- net SWDIO is gone; now on net YELLOW: U1.34 (PA13)
- net BLUE: no longer U1.32 (PA11)
- net GND: now also J2.5 (GND), J2.6 (Shield)
- net YELLOW: no longer U1.33 (PA12)
- new net USB_DM: J2.2 (D-), U1.32 (PA11)
- new net USB_DP: J2.3 (D+), U1.33 (PA12)
- no-connect marks 18 -> 20

Commit message: h7 initial
Parts:
- removed U1: STM32F411CEUx, Package_DFN_QFN:QFN-48-1EP_7x7mm_P0.5mm_EP5.6x5.6mm, symbol MCU_ST_STM32F4:STM32F411CEUx
- added U2: STM32H723VGTx, Package_QFP:LQFP-100_14x14mm_P0.5mm, symbol MCU_ST_STM32H7:STM32H723VGTx
- J4: footprint Connector_JST:JST_XH_B2B-XH-A_1x02_P2.50mm_Vertical -> Connector_PinHeader_1.27mm:PinHeader_1x02_P1.27mm_Vertical
Connections:
- net BOOT: now also U2.94 (BOOT0)
- net RESET1: now also U2.14 (NRST)
- net VMCU: now also U2.100 (VDD), U2.11 (VDD), U2.21 (VDDA), U2.27 (VDD), U2.50 (VDD), U2.6 (VBAT), U2.75 (VDD)
- net at Y2.1: now also U2.12 (PH0)
- net at Y2.3: now also U2.13 (PH1)
- new net: U2.10 (VSS), U2.26 (VSS), U2.49 (VSS), U2.74 (VSS), U2.99 (VSS)
- no-connect marks 20 -> 3
Other:
- moved on the sheet: C15, J2, R1

Commit message: h7 routing
Parts:
- removed J2: USB_B_Micro, Connector_USB:USB_Micro-B_Molex_47346-0001, symbol Connector:USB_B_Micro
- added C12: 2.2u, Capacitor_SMD:C_0201_0603Metric, symbol Device:C
- added C8: 100n, Capacitor_SMD:C_0201_0603Metric, symbol Device:C
- added J5: USB_C_Receptacle_USB2.0_16P, Connector_USB:USB_C_Receptacle_GCT_USB4110, symbol Connector:USB_C_Receptacle_USB2.0_16P
- added R10, R11: 5.1K, Resistor_SMD:R_0201_0603Metric, symbol Device:R
- C1, C23, C25, C4: footprint Capacitor_SMD:C_0603_1608Metric -> Capacitor_SMD:C_0201_0603Metric
- C10: footprint Capacitor_SMD:C_1206_3216Metric -> Capacitor_SMD:C_0402_1005Metric
- C11, C2, C21, C22, C24, C26: footprint Capacitor_SMD:C_0805_2012Metric -> Capacitor_SMD:C_0201_0603Metric
- C15: value 4.7u -> 2.2u; footprint Capacitor_SMD:C_1206_3216Metric -> Capacitor_SMD:C_0201_0603Metric
- C16, C3, C5, C6, C7, C9: footprint Capacitor_SMD:C_0402_1005Metric -> Capacitor_SMD:C_0201_0603Metric
- R7, R8: footprint Resistor_SMD:R_0603_1608Metric -> Resistor_SMD:R_0201_0603Metric
- R9: footprint Resistor_SMD:R_0402_1005Metric -> Resistor_SMD:R_0201_0603Metric
Connections:
- net GND: now also U2.10 (VSS), U2.19 (VSSA), U2.26 (VSS), U2.49 (VSS), U2.74 (VSS), U2.99 (VSS), C12.2, C8.2, J5.A1 (GND), J5.A12 (GND), J5.B1 (GND), J5.B12 (GND), J5.S1 (SHIELD), R10.2, R11.2
- net USB_DM: now also U2.70 (PA11), J5.A7 (D-), J5.B7 (D-)
- net USB_DP: now also U2.71 (PA12), J5.A6 (D+), J5.B6 (D+)
- net VMCU: now also C8.1
- net at C15.1: now also U2.48 (VCAP)
- net at U2.73 (VCAP): now also C12.1
- new net: J5.B8 (SBU2), R11.1
- new net: J5.A8 (SBU1), R10.1
- new net NOVBUS: J5.A4 (VBUS), J5.A9 (VBUS), J5.B4 (VBUS), J5.B9 (VBUS)
- no-connect marks 3 -> 1
Other:
- moved on the sheet: C15, C6, C7, C9, J1, R2

Commit message: h7 board almost full
Parts:
- removed R1: 10K, Resistor_SMD:R_0402_1005Metric, symbol Device:R
- J1: footprint Connector_PinHeader_2.54mm:PinHeader_1x04_P2.54mm_Vertical -> Connector_PinHeader_1.27mm:PinHeader_1x04_P1.27mm_Vertical
- J3: footprint Connector_JST:JST_XH_B5B-XH-A_1x05_P2.50mm_Vertical -> Connector_PinHeader_1.27mm:PinHeader_1x05_P1.27mm_Vertical
- R7, R8: footprint Resistor_SMD:R_0201_0603Metric -> Resistor_SMD:R_0402_1005Metric
Connections:
- net TX3 is gone; now on net U2RX: J1.4 (Pin_4)
- net BLUE: now also U2.15 (PC0)
- net GREEN: now also U2.7 (PC13)
- net MISO: now also U2.4 (PE5)
- net MOSI: now also U2.5 (PE6)
- net MOTOR0: now also J3.5 (Pin_5), U2.42 (PE12); no longer J3.2 (Pin_2)
- net MOTOR1: now also J3.4 (Pin_4), U2.43 (PE13); no longer J3.3 (Pin_3)
- net MOTOR2: now also J3.3 (Pin_3), U2.44 (PE14); no longer J3.4 (Pin_4)
- net MOTOR3: now also J3.2 (Pin_2), U2.45 (PE15); no longer J3.5 (Pin_5)
- net SCK: now also U2.1 (PE2)
- net YELLOW: now also U2.16 (PC1)
- net U2TX: now reaches U2.24 (PA2)
- net U2TX: now also J1.3 (Pin_3)
- net U2RX: now reaches U2.25 (PA3)
- net U2RX: now also R2.1
- removed net RX3: J1.3 (Pin_3), R2.1
