File: customboard/droneboardh7/droneboard.kicad_sch (KiCad schematic)
At the start: 62 parts, among them J1 Conn_01x04, J10 Conn_01x03_Pin, J2 Conn_01x04, J3 Conn_01x05_Pin, J4 Conn_01x02_Pin, J5 USB_C_Receptacle_USB2.0_16P, J6 Conn_01x04, SW1 SW_Push, SW2 SW_Push, U1 AP62300Z6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

Commit message: stuff
Parts:
- removed U2: STM32H723VGTx, Package_QFP:LQFP-100_14x14mm_P0.5mm, symbol MCU_ST_STM32H7:STM32H723VGTx
- added Q1: DMN2075U, Package_TO_SOT_SMD:SOT-23, symbol Transistor_FET:DMN2075U
- added R15: 10K, Resistor_SMD:R_0201_0603Metric, symbol Device:R
- added U2: STM32H743VGHx, Package_BGA:TFBGA-100_8x8mm_Layout10x10_P0.8mm, symbol MCU_ST_STM32H7:STM32H743VGHx
- added U3: LPS22HH, Package_LGA:ST_HLGA-10_2x2mm_P0.5mm_LayoutBorder3x2y, symbol Sensor_Pressure:LPS22HH
- C10: footprint Capacitor_SMD:C_0402_1005Metric -> Capacitor_SMD:C_0603_1608Metric
- C11: footprint Capacitor_SMD:C_0201_0603Metric -> Capacitor_SMD:C_0402_1005Metric
- J1, J2, J6: footprint Custom:PinHeaderWide4x -> Connector_PinHeader_2.54mm:PinHeader_1x04_P2.54mm_Vertical
Connections:
- net BLUE: now also U2.A1 (PC14)
- net BOOT: now also U2.D5 (BOOT0)
- net GND: now also Q1.2 (S), R15.1, U2.C2 (VSS), U2.E4 (VSS), U2.E5 (VSS), U2.E6 (VSS), U2.G1 (VSSA), U2.J1 (VSS), U3.3 (GND), U3.5 (SA0), U3.8 (GND), U3.9 (GND); no longer J2.2 (Pin_2)
- net GREEN: now also U2.A2 (PC13)
- net IMU_CS: now also U2.A5 (PB7)
- net MISO: now also U2.A6 (PB4)
- net MOSI: now also U2.C5 (PB5)
- net MOTOR0: now also U2.J7 (PB10)
- net MOTOR1: now also U2.K7 (PB11)
- net MOTOR2: now also U2.K8 (PB12)
- net MOTOR3: now also U2.J8 (PB13)
- net RESET1: now also U2.E1 (NRST)
- net SCK: now also U2.A7 (PB3)
- net SWCLK: now also U2.A9 (PA14)
- net SWDIO: now also U2.A10 (PA13)
- net U2RX: now also U2.K2 (PA3)
- net U2TX: now also U2.J2 (PA2)
- net U4RX: now also U2.H2 (PA1)
- net U4TX: now also U2.G2 (PA0)
- net U7RX: now also U2.H5 (PE7)
- net U7TX: now also U2.J5 (PE8)
- net USB_DM: now also U2.C10 (PA11)
- net USB_DP: now also U2.B10 (PA12)
- net VBATMON: now also U2.F3 (PC3_C), U2.G3 (PA4)
- net VMCU: now also U2.B2 (VBAT), U2.D2 (VDD), U2.F4 (VDDLDO), U2.F5 (VDD), U2.F6 (VDD33_USB), U2.H1 (VDDA), U2.K1 (VDD), U3.1 (Vdd_IO), U3.10 (VDD), U3.6 (~{CS})
- net YELLOW: now also U2.B1 (PC15)
- net at Y2.1: now also U2.C1 (PH0)
- net at Y2.3: now also U2.D1 (PH1)
- net at C12.1: now also U2.F8 (VCAP)
- net at C15.1: now also U2.E7 (VCAP)
- new net: J2.2 (Pin_2), Q1.3 (D)
- new net BARO_SCL: U2.K10 (PD12), U3.2 (SCL)
- new net BARO_SDA: U2.J10 (PD13), U3.4 (SDA)
- new net VTX_PWR: Q1.1 (G), R15.2, U2.F1 (PC0)
- no-connect marks 62 -> 55

Commit message: 743 further work
Parts:
- added C19: 100n, Capacitor_SMD:C_0201_0603Metric, symbol Device:C
Connections:
- net GND: now also C19.1; no longer U3.5 (SA0)
- net VMCU: now also C19.2; no longer U3.6 (~{CS})
- net BARO_MOSI: now reaches U2.G7 (PE14)
- net BARO_MOSI: now also U3.4 (SDA)
- net BARO_SCK: now reaches U2.J6 (PE12)
- net BARO_SCK: now also U3.2 (SCL)
- net BARO_MISO: now reaches U2.K6 (PE13)
- net BARO_MISO: now also U3.5 (SA0)
- net BARO_CS: now reaches U2.K9 (PD8)
- net BARO_CS: now also U3.6 (~{CS})
- net BARO_SCL: no longer names the net of U2.K10 (PD12)
- net BARO_SCL: no longer U3.2 (SCL)
- net BARO_SDA: no longer names the net of U2.J10 (PD13)
- net BARO_SDA: no longer U3.4 (SDA)
- no-connect marks 55 -> 56

Commit message: move mcu
Parts:
- removed Q1: DMN2075U, Package_TO_SOT_SMD:SOT-23, symbol Transistor_FET:DMN2075U
- added Q1: DMN2056U, Package_TO_SOT_SMD:SOT-23, symbol Transistor_FET:DMN2056U
- SW1, SW2: value SW_Push -> KMR221NGLFS; footprint Button_Switch_THT:SW_PUSH_1P1T_6x3.5mm_H4.3_APEM_MJTP1243 -> Button_Switch_SMD:SW_Push_1P1T_NO_CK_KMR2
Connections:
- net GND: now also Q1.2 (S)
- net IMU_CS: now also U2.A4 (PB9); no longer U2.A5 (PB7)
- net VMCU: now also U2.F7 (PDR_ON)
- net VTX_PWR: now also Q1.1 (G)
- net at J2.2 (Pin_2): now also Q1.3 (D)
Changed lines of the file:
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@@
 	)
 	(no_connect
+		(at 187.96 120.65)
+	)
+	(no_connect
 		(at 156.21 184.15)
 	)
@@
 	)
 	(no_connect
-		(at 109.22 135.89)
-	)
-	(no_connect
 		(at 109.22 113.03)
 	)
@@
 	(wire
 		(pts
+			(xy 49.53 80.01) (xy 63.5 80.01)
+		)
+		(stroke
+			(width 0)
+			(type default)
+		)
+	)
+	(wire
+		(pts
 			(xy 232.41 110.49) (xy 228.6 110.49)
 		)
@@
 	(wire
 		(pts
-			(xy 109.22 130.81) (xy 118.11 130.81)
+			(xy 109.22 135.89) (xy 118.11 135.89)
 		)
 		(stroke
@@
 	)
 	(label "IMU_CS"
-		(at 118.11 130.81 180)
+		(at 118.11 135.89 180)
 		(effects
 			(font
@@
 		)
 	)
+	(label "VMCU"
+		(at 49.53 80.01 0)
+		(effects
+			(font
+				(size 1.27 1.27)
+			)
+			(justify left bottom)
+		)
+	)
 	(label "U4TX"
 		(at 118.11 69.85 180)
@@
 			)
 		)
-		(property "Value" "SW_Push"
+		(property "Value" "KMR221NGLFS"
 			(at 64.77 58.42 0)
 			(effects
@@
 			)
 		)
-		(property "Footprint" "Button_Switch_THT:SW_PUSH_1P1T_6x3.5mm_H4.3_APEM_MJTP1243"
+		(property "Footprint" "Button_Switch_SMD:SW_Push_1P1T_NO_CK_KMR2"
 			(at 64.77 58.42 0)
 			(effects
@@
 	)
 	(symbol
+		(lib_id "Transistor_FET:DMN2056U")
+		(at 57.15 231.14 0)
+		(unit 1)
+		(exclude_from_sim no)
+		(in_bom yes)
+		(on_board yes)
+		(dnp no)
+		(fields_autoplaced yes)
+		(property "Reference" "Q1"
+			(at 63.5 229.8699 0)
+			(effects
+				(font
+					(size 1.27 1.27)
+				)
+				(justify left)
+			)
+		)
+		(property "Value" "DMN2056U"
+			(at 63.5 232.4099 0)
+			(effects
+				(font
+					(size 1.27 1.27)
+				)
+				(justify left)
+			)
+		)
+		(property "Footprint" "Package_TO_SOT_SMD:SOT-23"
+			(at 62.23 233.045 0)
+			(effects
+				(font
+					(size 1.27 1.27)
+					(italic yes)
+				)
+				(justify left)
+				(hide yes)
+			)
+		)
+		(property "Datasheet" "http://www.diodes.com/assets/Datasheets/DMN2056U.pdf"
+			(at 62.23 234.95 0)
+			(effects
+				(font
+					(size 1.27 1.27)
+				)
+				(justify left)
+				(hide yes)
+			)
+		)
+		(property "Description" "4A Id, 20V Vds, N-Channel MOSFET, SOT-23"
+			(at 57.15 231.14 0)
+			(effects
+				(font
+					(size 1.27 1.27)
+				)
+				(hide yes)
+			)
+		)
+		(pin "2"
+		)
+		(pin "3"
+		)
+		(pin "1"
+		)
+		(instances
+			(project ""
+				(path "/04179b3e-2b25-41d4-a9af-8911a5c82cad"
+					(reference "Q1")
+					(unit 1)
+				)
+			)
+		)
+	)
+	(symbol
 		(lib_id "Device:C")
 		(at 43.18 187.96 0)
@@
 			)
 		)
-		(property "Value" "SW_Push"
+		(property "Value" "KMR221NGLFS"
 			(at 46.99 57.15 0)
 			(effects
@@
 			)
 		)
-		(property "Footprint" "Button_Switch_THT:SW_PUSH_1P1T_6x3.5mm_H4.3_APEM_MJTP1243"
+		(property "Footprint" "Button_Switch_SMD:SW_Push_1P1T_NO_CK_KMR2"
 			(at 46.99 57.15 0)
 			(effects
@@
 					(unit 1)
 				)
-			)
-		)
-	)
-	(symbol
-		(lib_id "Transistor_FET:DMN2075U")
-		(at 57.15 231.14 0)
-		(unit 1)
-		(exclude_from_sim no)
-		(in_bom yes)
-		(on_board yes)
-		(dnp no)
-		(fields_autoplaced yes)
-		(property "Reference" "Q1"
-			(at 63.5 229.8699 0)
-			(effects
-				(font
-					(size 1.27 1.27)
-				)
-				(justify left)
-			)
-		)
-		(property "Value" "DMN2075U"
-			(at 63.5 232.4099 0)
-			(effects
-				(font
-					(size 1.27 1.27)
-				)
-				(justify left)
-			)
-		)
-		(property "Footprint" "Package_TO_SOT_SMD:SOT-23"
-			(at 62.23 233.045 0)
-			(effects
-				(font
-					(size 1.27 1.27)
-					(italic yes)
-				)
-				(justify left)
-				(hide yes)
-			)
-		)
-		(property "Datasheet" "http://www.diodes.com/assets/Datasheets/DMN2075U.pdf"
-			(at 62.23 234.95 0)
-			(effects
-				(font
-					(size 1.27 1.27)
-				)
-				(justify left)
-				(hide yes)
-			)
-		)
-		(property "Description" "4.2A Id, 20V Vds, N-Channel MOSFET, SOT-23"
-			(at 57.15 231.14 0)
-			(effects
-				(font
-					(size 1.27 1.27)
-				)
-				(hide yes)
-			)
-		)
-		(pin "1"
-		)
-		(pin "3"
-		)
-		(pin "2"
-		)
-		(instances
-			(project ""
-				(path "/04179b3e-2b25-41d4-a9af-8911a5c82cad"
-					(reference "Q1")
-					(unit 1)
-				)
