File: customboard/droneboardh7/droneboard.kicad_pcb (KiCad board)
At the start: 4 copper layers, 38 x 38 mm, 62 parts, among them J1 Conn_01x04, J10 Conn_01x03_Pin, J2 Conn_01x04, J3 Conn_01x05_Pin, J4 Conn_01x02_Pin, J5 USB_C_Receptacle_USB2.0_16P, J6 Conn_01x04, SW1 SW_Push, SW2 SW_Push, U1 AP62300Z6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

Commit message: stuff
Parts:
- added Q1: DMN2075U, Package_TO_SOT_SMD:SOT-23, F.Cu at (55.9, 106.4)
- added R15: 10K, Resistor_SMD:R_0201_0603Metric, F.Cu at (60.5, 106.9)
- added U3: LPS22HH, Package_LGA:ST_HLGA-10_2x2mm_P0.5mm_LayoutBorder3x2y, F.Cu at (67.8, 105.9)
- C10: footprint Capacitor_SMD:C_0402_1005Metric -> Capacitor_SMD:C_0603_1608Metric
- C11: footprint Capacitor_SMD:C_0201_0603Metric -> Capacitor_SMD:C_0402_1005Metric
- C12, C15, C3, C5, C6, C7, C8, C9, R1, R12, R2: moved to B.Cu
- J1, J2, J6: footprint Custom:PinHeaderWide4x -> Connector_PinHeader_2.54mm:PinHeader_1x04_P2.54mm_Vertical
- U2: value STM32H723VGTx -> STM32H743VGHx; footprint Package_QFP:LQFP-100_14x14mm_P0.5mm -> Package_BGA:TFBGA-100_8x8mm_Layout10x10_P0.8mm
- moved C7 16.7 mm to (74.6, 102.8), turned to 90 degrees
- moved C15 13.1 mm to (75.4, 102.0), turned to 90 degrees
- moved C6 12.4 mm to (70.6, 104.4), turned to 90 degrees
- moved C5 11.6 mm to (70.6, 106.0), turned to 90 degrees
- moved C9 11.1 mm to (73.8, 102.8), turned to 90 degrees
- moved C3 10.7 mm to (71.4, 101.2), turned to 90 degrees
- moved C16 10.1 mm to (68.5, 103.5)
- moved Y2 9.92 mm to (68.0, 101.3)
- moved J1 9.28 mm to (59.7, 114.3)
- moved C24 9.00 mm to (61.8, 99.4), turned to 0 degrees
- moved C25 8.84 mm to (65.9, 101.5), turned to 180 degrees
- moved R9 8.41 mm to (79.7, 94.7), turned to 180 degrees
- moved C11 8.31 mm to (68.7, 98.3), turned to -90 degrees
- moved U6 7.73 mm to (64.6, 99.4), turned to 0 degrees
- moved C10 7.24 mm to (67.4, 97.7), turned to -90 degrees
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Connections:
- J2 pad 2: /GND -> Net-(J2-Pin_2)
Routing:
- net /GND: track 198.2 -> 31.3 mm, vias 37 -> 14
- net /VMCU: track 51.6 -> 31.1 mm, vias 13 -> 15
- net /5V: track 78.1 -> 98.0 mm, vias 7 -> 9
- net /VTX_PWR: track 0.00 -> 15.5 mm
- net /BARO_SCL: track 0.00 -> 15.4 mm, vias 0 -> 2
- net /BARO_SDA: track 0.00 -> 12.8 mm, vias 0 -> 2
- net /GREEN: track 5.06 -> 17.0 mm, vias 0 -> 2
- net /U7RX: track 7.70 -> 19.3 mm
- net /BLUE: track 4.83 -> 15.5 mm, vias 0 -> 2
- net /YELLOW: track 5.81 -> 15.2 mm, vias 0 -> 2
- net /MOTOR0: track 5.50 -> 14.6 mm
- net /U4RX: track 10.4 -> 19.2 mm
- net /U7TX: track 6.63 -> 15.4 mm
- net /BOOT: track 22.4 -> 14.2 mm, vias 2 -> 1
- net /MOTOR1: track 4.92 -> 13.0 mm
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Other:
- board text removed: "2"
- board text removed: "4"
- board text removed: "5"
- board text removed: "7"
- board text removed: "G"
- board text removed: "T"

Commit message: 743 further work
Parts:
- added C19: 100n, Capacitor_SMD:C_0201_0603Metric, B.Cu at (72.2, 108.9)
- U3: moved to B.Cu
- moved U3 6.73 mm to (74.0, 108.6)
- moved C24 0.49 mm to (61.3, 99.4)
- moved U6 0.38 mm to (64.2, 99.4)
- moved Y2 0.07 mm to (68.0, 101.3)
Connections:
- U2 pad G7: unconnected-(U2-PE14-PadG7) -> /BARO_MOSI
- U2 pad J10: /BARO_SDA -> unconnected-(U2-PD13-PadJ10)
- U2 pad J6: unconnected-(U2-PE12-PadJ6) -> /BARO_SCK
- U2 pad K10: /BARO_SCL -> unconnected-(U2-PD12-PadK10)
- U2 pad K6: unconnected-(U2-PE13-PadK6) -> /BARO_MISO
- U2 pad K9: unconnected-(U2-PD8-PadK9) -> /BARO_CS
- U3 pad 2: /BARO_SCL -> /BARO_SCK
- U3 pad 4: /BARO_SDA -> /BARO_MOSI
- U3 pad 5: /GND -> /BARO_MISO
- U3 pad 6: /VMCU -> /BARO_CS
Routing:
- net /5V: track 98.0 -> 20.2 mm
- net /BARO_SCL: track 15.4 -> 0.00 mm, vias 2 -> 0
- net /BARO_SDA: track 12.8 -> 0.00 mm, vias 2 -> 0
- net /VMCU: track 31.1 -> 25.7 mm, vias 15 -> 14
- net /BARO_MOSI: track 0.00 -> 4.41 mm, vias 0 -> 1
- net /BARO_SCK: track 0.00 -> 4.01 mm, vias 0 -> 1
- net /BARO_CS: track 0.00 -> 3.62 mm, vias 0 -> 1
- net Net-(D2-A): track 0.00 -> 1.71 mm
- net /BARO_MISO: track 0.00 -> 1.48 mm, vias 0 -> 1
- net Net-(D1-A): track 0.00 -> 1.28 mm
- net /GND: track 31.3 -> 32.5 mm, vias 14 -> 23
- net Net-(D3-A): track 0.00 -> 1.20 mm
- net Net-(D4-A): track 0.00 -> 1.18 mm
- net /VGYRO: track 12.9 -> 13.8 mm

Commit message: move mcu
Parts:
- Q1: value DMN2075U -> DMN2056U
- SW1, SW2: value SW_Push -> KMR221NGLFS; footprint Button_Switch_THT:SW_PUSH_1P1T_6x3.5mm_H4.3_APEM_MJTP1243 -> Button_Switch_SMD:SW_Push_1P1T_NO_CK_KMR2
- moved SW1 14.5 mm to (84.3, 96.4), turned to 180 degrees
- moved C19 6.08 mm to (73.7, 114.8), turned to 180 degrees
- moved SW2 5.03 mm to (84.4, 92.5)
- moved C26 4.68 mm to (68.7, 100.6), turned to 90 degrees
- moved C12 4.66 mm to (76.9, 107.9)
- moved C16 4.66 mm to (68.8, 108.2)
- moved C9 4.66 mm to (74.1, 107.5)
- moved U3 4.66 mm to (74.2, 113.2)
- moved C15 4.66 mm to (75.7, 106.7)
- moved C3 4.66 mm to (71.7, 105.8)
- moved C5 4.66 mm to (70.9, 110.6)
- moved C6 4.66 mm to (70.9, 109.0)
- moved C7 4.66 mm to (74.9, 107.5)
- moved C8 4.66 mm to (73.3, 107.5)
- moved U2 4.66 mm to (74.5, 107.5)
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Connections:
- U2 pad A4: unconnected-(U2-PB9-PadA4) -> /IMU_CS
- U2 pad A5: /IMU_CS -> unconnected-(U2-PB7-PadA5)
- U2 pad F7: unconnected-(U2-PDR_ON-PadF7) -> /VMCU
Routing:
- net /5V: track 20.2 -> 38.2 mm, vias 9 -> 8
- net /BOOT: track 14.2 -> 23.8 mm, vias 1 -> 2
- net /RESET1: track 17.4 -> 25.7 mm, vias 1 -> 2
- net /MISO: track 6.90 -> 11.7 mm
- net /SWDIO: track 8.28 -> 13.0 mm
- net /SWCLK: track 5.41 -> 10.2 mm
- net /MOSI: track 8.29 -> 13.1 mm
- net /MOTOR1: track 13.0 -> 8.47 mm
- net /MOTOR2: track 12.5 -> 7.97 mm
- net /MOTOR3: track 12.8 -> 8.28 mm
- net /MOTOR0: track 14.6 -> 10.1 mm
- net /VBATMON: track 23.3 -> 27.2 mm
- net /U7RX: track 19.3 -> 15.6 mm
- net /U2TX: track 10.7 -> 7.49 mm
- net /SCK: track 9.22 -> 12.5 mm
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- added copper zone on F.Cu, net /VMCU

Commit message: minor fixes
Parts:
- Y2: value CSTNE20M0V53Z000R0 -> CSTNE8M00G520000R0
- moved C22 0.30 mm to (71.3, 90.2)
- moved Y2 0.08 mm to (68.3, 105.9)
Routing:
- net /GND: track 31.3 -> 28.7 mm, vias 31 -> 35
- net /5V: track 38.2 -> 39.4 mm
Other:
- board text added: "2"
- board text added: "4"
- board text added: "5"
- board text added: "7"
- board text added: "G"
- board text added: "T"
