File: customboard/droneboardh7/droneboard.kicad_pcb (KiCad board)
At the start: 4 copper layers, 38 x 38 mm, 62 parts, among them J1 Conn_01x04, J10 Conn_01x03_Pin, J2 Conn_01x04, J3 Conn_01x05_Pin, J4 Conn_01x02_Pin, J5 USB_C_Receptacle_USB2.0_16P, J6 Conn_01x04, SW1 SW_Push, SW2 SW_Push, U1 AP62300Z6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

Commit message: stuff
Parts:
- removed U2: STM32H723VGTx, Package_QFP:LQFP-100_14x14mm_P0.5mm
- added U3: STM32H743VITx, Package_QFP:LQFP-100_14x14mm_P0.5mm, F.Cu at (69.0, 105.9)
Routing:
- net /VMCU: track 51.6 -> 54.6 mm

Commit message: stuff
Parts:
- removed R12, R2: 10K, Resistor_SMD:R_0201_0603Metric
- added Q1: DMN2056U, Package_TO_SOT_SMD:SOT-23, F.Cu at (58.2, 99.0)
- J1, J2, J6: footprint Custom:PinHeaderWide4x -> Connector_JST:JST_SH_SM04B-SRSS-TB_1x04-1MP_P1.00mm_Horizontal
- J3: value Conn_01x05_Pin -> Conn_01x08_MountingPin; footprint Connector_PinHeader_2.00mm:PinHeader_1x05_P2.00mm_Vertical -> Connector_JST:JST_SH_SM08B-SRSS-TB_1x08-1MP_P1.00mm_Horizontal
- J4: value Conn_01x02_Pin -> Conn_01x08_MountingPin; footprint Connector_PinHeader_2.54mm:PinHeader_1x02_P2.54mm_Vertical -> Connector_JST:JST_SH_SM08B-SRSS-TB_1x08-1MP_P1.00mm_Horizontal; moved to B.Cu
- R7, R8: moved to B.Cu
- SW1, SW2: footprint Button_Switch_THT:SW_PUSH_1P1T_6x3.5mm_H4.3_APEM_MJTP1243 -> Button_Switch_SMD:SW_Push_1P1T-SH_NO_CK_KMR2xxG
- moved J4 29.7 mm to (72.2, 116.8)
- moved R8 22.3 mm to (67.2, 106.8)
- moved R7 22.2 mm to (70.3, 106.8), turned to 180 degrees
- moved C13 13.4 mm to (53.2, 109.5), turned to 90 degrees
- moved R13 13.0 mm to (57.5, 109.6), turned to 90 degrees
- moved R14 12.4 mm to (59.0, 108.5), turned to 0 degrees
- moved R9 11.6 mm to (81.8, 91.2), turned to -90 degrees
- moved C14 10.6 mm to (60.0, 106.4), turned to 90 degrees
- moved R1 10.6 mm to (60.3, 99.2)
- moved C18 9.08 mm to (51.7, 105.5), turned to -90 degrees
- moved U1 8.77 mm to (56.7, 107.6), turned to 0 degrees
- moved D1 6.64 mm to (53.2, 95.7)
- moved D3 6.64 mm to (53.2, 92.4)
- moved D4 6.64 mm to (53.2, 94.0)
- moved R3 6.64 mm to (55.8, 95.7)
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Connections:
- J2 pad 2: /GND -> Net-(J2-Pin_2)
- J3 pad 1: /GND -> /12V
- J3 pad 2: /MOTOR3 -> /GND
- J3 pad 3: /MOTOR2 -> unconnected-(J3-Pin_3-Pad3)
- J3 pad 4: /MOTOR1 -> unconnected-(J3-Pin_4-Pad4)
- R1 pad 1: /U4RX -> /VTX_PWR
- R1 pad 2: /VMCU -> /GND
- U3 pad 4: unconnected-(U3-PE5-Pad4) -> /VTX_PWR
Routing:
- net /GND: track 198.2 -> 117.8 mm, vias 37 -> 46
- net /12V: track 8.24 -> 40.4 mm, vias 0 -> 3
- net /VBATMON: track 30.8 -> 8.07 mm, vias 2 -> 1
- net /VMCU: track 54.6 -> 43.4 mm, vias 13 -> 12
- net /RESET1: track 22.5 -> 30.1 mm, vias 1 -> 2
- net /MOTOR3: track 6.57 -> 12.0 mm, vias 0 -> 1
- net /MOTOR1: track 4.92 -> 9.78 mm, vias 0 -> 1
- net Net-(J2-Pin_2): track 0.00 -> 4.31 mm
- net /5V: track 78.1 -> 81.9 mm, vias 7 -> 14
- net /VTX_PWR: track 0.00 -> 3.60 mm
- net /GREEN: track 5.06 -> 8.52 mm
- net /YELLOW: track 5.81 -> 9.11 mm
- net /BLUE: track 4.83 -> 7.80 mm
- net /U4RX: track 10.4 -> 13.0 mm, vias 2 -> 0
- net /BOOT: track 22.4 -> 24.7 mm
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Other:
- board text added: "M"
- board text removed: "BAT"
- board text removed: "M0"

Commit message: stuff
Other:
- board text added: "UART2"
- board text added: "UART4"
- board text added: "UART7"
- board text removed: "2"
- board text removed: "4"
- board text removed: "7"
Changed lines of the file:
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@@
 			)
 		)
+		(model "${KIPRJMOD}/components/3dmodels/KMR221GLFS--3DModel-STEP-56544.STEP"
+			(offset
+				(xyz 0 0 1.5)
+			)
+			(scale
+				(xyz 1 1 1)
+			)
+			(rotate
+				(xyz -90 -0 -0)
+			)
+		)
 	)
 	(footprint "Capacitor_SMD:C_0201_0603Metric"
@@
 		(tags "connector JST SH horizontal")
 		(property "Reference" "J2"
-			(at 2.01 -3.86 90)
+			(at 2.65 -2.57 90)
 			(layer "F.SilkS")
 			(effects
@@
 			)
 		)
+		(model "${KIPRJMOD}/components/3dmodels/SM04B-SRSS-TB_LF__SN_.stp"
+			(offset
+				(xyz 0 1.25 -0.3)
+			)
+			(scale
+				(xyz 1 1 1)
+			)
+			(rotate
+				(xyz -90 -0 -0)
+			)
+		)
 	)
 	(footprint "Connector_PinHeader_2.54mm:PinHeader_1x03_P2.54mm_Vertical"
@@
 			)
 		)
+		(model "${KIPRJMOD}/components/3dmodels/USB4110GFA--3DModel-STEP-269445.STEP"
+			(offset
+				(xyz 0 2.5 0)
+			)
+			(scale
+				(xyz 1 1 1)
+			)
+			(rotate
+				(xyz -90 -0 -0)
+			)
+		)
 	)
 	(footprint "Capacitor_SMD:C_0201_0603Metric"
@@
 		(tags "resistor")
 		(property "Reference" "R3"
-			(at -1.825 0 0)
+			(at -1.725 0.44 0)
 			(layer "F.SilkS")
 			(effects
@@
 		(tags "SOT TO_SOT_SMD")
 		(property "Reference" "Q1"
-			(at 1.73 1.13 90)
+			(at -2.51 0.02 180)
 			(layer "F.SilkS")
 			(effects
@@
 		(tags "connector JST SH horizontal")
 		(property "Reference" "J1"
-			(at 0 -3.98 90)
+			(at 2.59 -2.51 90)
 			(layer "F.SilkS")
 			(effects
@@
 			)
 		)
+		(model "${KIPRJMOD}/components/3dmodels/SM04B-SRSS-TB_LF__SN_.stp"
+			(offset
+				(xyz 0 1.25 -0.3)
+			)
+			(scale
+				(xyz 1 1 1)
+			)
+			(rotate
+				(xyz -90 -0 -0)
+			)
+		)
 	)
 	(footprint "Crystal:Resonator_SMD_Murata_CSTxExxV-3Pin_3.0x1.1mm"
@@
 			)
 		)
+		(model "${KIPRJMOD}/components/3dmodels/KMR221GLFS--3DModel-STEP-56544.STEP"
+			(offset
+				(xyz 0 0 1.4)
+			)
+			(scale
+				(xyz 1 1 1)
+			)
+			(rotate
+				(xyz -90 -0 -0)
+			)
+		)
 	)
 	(footprint "Resistor_SMD:R_0402_1005Metric"
@@
 			)
 		)
+		(model "${KIPRJMOD}/components/3dmodels/SM04B-SRSS-TB_LF__SN_.stp"
+			(offset
+				(xyz 0 1.25 -0.3)
+			)
+			(scale
+				(xyz 1 1 1)
+			)
+			(rotate
+				(xyz -90 -0 -0)
+			)
+		)
 	)
 	(footprint "LED_SMD:LED_0603_1608Metric"
@@
 			)
 		)
+		(model "${KIPRJMOD}/components/3dmodels/SM08B-SRSS-TB (LF)(SN)--3DModel-STEP-269445.STEP"
+			(offset
+				(xyz 0 -2.5 1.5)
+			)
+			(scale
+				(xyz 1 1 1)
+			)
+			(rotate
+				(xyz -90 -0 -0)
+			)
+		)
 	)
 	(footprint "Package_TO_SOT_SMD:SOT-563"
@@
 			)
 		)
+		(model "${KIPRJMOD}/components/3dmodels/SM08B-SRSS-TB (LF)(SN)--3DModel-STEP-269445.STEP"
+			(offset
+				(xyz 0 -2.5 1.5)
+			)
+			(scale
+				(xyz 1 1 1)
+			)
+			(rotate
+				(xyz -90 -0 -0)
+			)
+		)
 	)
 	(footprint "Resistor_SMD:R_0402_1005Metric"
@@
 		(layer "Edge.Cuts")
 	)
+	(gr_text "5"
+		(at 55.18 98.19 0)
+		(layer "F.SilkS")
+		(effects
+			(font
+				(size 0.8 0.8)
+				(thickness 0.15)
+			)
+			(justify left bottom)
+		)
+	)
+	(gr_text "G"
+		(at 56.17 108.24 0)
+		(layer "F.SilkS")
+		(effects
+			(font
+				(size 0.8 0.8)
+				(thickness 0.15)
+			)
+			(justify left bottom)
+		)
+	)
 	(gr_text "R"
 		(at 87.6 113.02 90)
@@
 		)
 	)
+	(gr_text "R"
+		(at 56.22 109.29 0)
+		(layer "F.SilkS")
+		(effects
+			(font
+				(size 0.8 0.8)
+				(thickness 0.15)
+			)
+			(justify left bottom)
+		)
+	)
+	(gr_text "T"
+		(at 56.36 110.36 0)
+		(layer "F.SilkS")
+		(effects
+			(font
+				(size 0.8 0.8)
+				(thickness 0.15)
+			)
+			(justify left bottom)
+		)
+	)
 	(gr_text "+"
 		(at 68.16 113.91 0)
@@
 		)
 	)
-	(gr_text "2"
-		(at 55.24 111.83 0)
+	(gr_text "UART2"
+		(at 52.14 112.44 0)
+		(layer "F.SilkS")
+		(effects
+			(font
+				(size 0.8 0.8)
+				(thickness 0.15)
+			)
+			(justify left bottom)
+		)
+	)
+	(gr_text "R"
+		(at 56.06 101.39 0)
 		(layer "F.SilkS")
 		(effects
@@
 		)
 	)
-	(gr_text "7"
-		(at 60.58 112.35 0)
+	(gr_text "UART7"
+		(at 59.1 117.5 90)
+		(layer "F.SilkS")
+		(effects
+			(font
+				(size 0.8 0.8)
+				(thickness 0.15)
+			)
+			(justify left bottom)
+		)
+	)
+	(gr_text "5"
+		(at 56.21 107.22 0)
 		(layer "F.SilkS")
 		(effects
@@
 		)
 	)
-	(gr_text "4"
-		(at 56.5 104.25 0)
+	(gr_text "UART4"
+		(at 50.87 104.84 0)
 		(layer "F.SilkS")
 		(effects
@@
 		(layer "F.SilkS")
 		(effects
+			(font
+				(size 0.8 0.8)
+				(thickness 0.15)
+			)
+			(justify left bottom)
+		)
+	)
+	(gr_text "T"
+		(at 56.18 102.51 0)
+		(layer "F.SilkS")
+		(effects

Commit message: stuff
Parts:
- C10: footprint Capacitor_SMD:C_0402_1005Metric -> Capacitor_SMD:C_0603_1608Metric
- J1, J2, J6: value Conn_01x04 -> Conn_01x04_MountingPin
- SW1, SW2: value SW_Push -> KMR221GLFS
- Y2: value CSTNE20M0V53Z000R0 -> CSTNE8M00G520000R0
- moved C3 2.99 mm to (64.4, 94.3), turned to 0 degrees
- moved C25 1.76 mm to (58.5, 92.7), turned to 0 degrees
- moved C11 0.86 mm to (62.1, 96.1)
- moved C10 0.22 mm to (61.2, 94.7)
- moved C26 0.20 mm to (61.3, 93.4)
Routing:
- net /GND: track 117.8 -> 110.0 mm, vias 46 -> 52
- net /5V: track 81.9 -> 88.6 mm, vias 14 -> 16
- net /VMCU: track 43.4 -> 43.1 mm, vias 12 -> 14
