File: customboard/droneboardh743_bga/droneboard.kicad_sch (KiCad schematic)
At the start: 68 parts, among them J1 Conn_01x04_MountingPin, J10 Conn_01x03_Pin, J2 Conn_01x04_MountingPin, J3 Conn_01x08_MountingPin, J4 Conn_01x08_MountingPin, J5 USB_C_Receptacle_USB2.0_16P, J6 Conn_01x06_MountingPin, J7 Conn_01x06_MountingPin, Q1 DMN3042L, SW1 434133025816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

Commit message: HAL fixes, remove 5V diode
Parts:
- removed D5: MBR120VLSFT1G, Diode_SMD:D_SOD-123F, symbol Diode:MBR1020VL
Connections:
- net 5V: now also C22.1, C24.1, J2.1 (Pin_1), R4.1, U5.1 (IN), U5.3 (EN), U6.1 (IN), U6.3 (EN)
- removed net VUSB: C22.1, C24.1, J2.1 (Pin_1), J5.A4 (VBUS), J5.A9 (VBUS), J5.B4 (VBUS), J5.B9 (VBUS), R4.1, U5.1 (IN), U5.3 (EN), U6.1 (IN), U6.3 (EN)
- new net NOVBUS: J5.A4 (VBUS), J5.A9 (VBUS), J5.B4 (VBUS), J5.B9 (VBUS)
Changed lines of the file:
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@@
 	(paper "A1")
 	(junction
+		(at 72.39 237.49)
+		(diameter 0)
+		(color 0 0 0 0)
+	)
+	(junction
 		(at 228.6 120.65)
 		(diameter 0)
@@
 	(wire
 		(pts
-			(xy 405.13 35.56) (xy 416.56 35.56)
+			(xy 72.39 237.49) (xy 166.37 237.49)
 		)
 		(stroke
@@
 	(wire
 		(pts
-			(xy 275.59 144.78) (xy 266.7 144.78)
-		)
-		(stroke
-			(width 0)
-			(type default)
-		)
-	)
-	(wire
-		(pts
 			(xy 109.22 146.05) (xy 125.73 146.05)
 		)
@@
 	(wire
 		(pts
-			(xy 424.18 35.56) (xy 441.96 35.56)
-		)
-		(stroke
-			(width 0)
-			(type default)
-		)
-	)
-	(wire
-		(pts
 			(xy 109.22 148.59) (xy 125.73 148.59)
 		)
@@
 	(wire
 		(pts
-			(xy 40.64 237.49) (xy 166.37 237.49)
+			(xy 40.64 237.49) (xy 72.39 237.49)
 		)
 		(stroke
@@
 	(wire
 		(pts
-			(xy 156.21 153.67) (xy 163.83 153.67)
-		)
-		(stroke
-			(width 0)
-			(type default)
-		)
-	)
-	(wire
-		(pts
 			(xy 19.05 41.91) (xy 19.05 82.55)
 		)
@@
 	(wire
 		(pts
+			(xy 72.39 237.49) (xy 72.39 242.57)
+		)
+		(stroke
+			(width 0)
+			(type default)
+		)
+	)
+	(wire
+		(pts
 			(xy 113.03 41.91) (xy 123.19 41.91)
 		)
@@
 	(wire
 		(pts
+			(xy 266.7 144.78) (xy 275.59 144.78)
+		)
+		(stroke
+			(width 0)
+			(type default)
+		)
+	)
+	(wire
+		(pts
 			(xy 109.22 90.17) (xy 125.73 90.17)
 		)
@@
 	(wire
 		(pts
-			(xy 63.5 242.57) (xy 72.39 242.57)
-		)
-		(stroke
-			(width 0)
-			(type default)
-		)
-	)
-	(wire
-		(pts
 			(xy 109.22 189.23) (xy 125.73 189.23)
 		)
@@
 		)
 	)
-	(label "VUSB"
-		(at 163.83 153.67 180)
+	(label "GND"
+		(at 172.72 40.64 0)
 		(effects
 			(font
 				(size 1.27 1.27)
 			)
-			(justify right bottom)
+			(justify left bottom)
 		)
 	)
-	(label "GND"
-		(at 172.72 40.64 0)
+	(label "NOVBUS"
+		(at 156.21 153.67 0)
 		(effects
 			(font
@@
 		)
 	)
-	(label "VUSB"
+	(label "5V"
 		(at 245.11 53.34 0)
 		(effects
@@
 		)
 	)
-	(label "VUSB"
-		(at 63.5 242.57 0)
-		(effects
-			(font
-				(size 1.27 1.27)
-			)
-			(justify left bottom)
-		)
-	)
 	(label "GREEN"
 		(at 181.61 198.12 0)
@@
 		)
 	)
-	(label "VUSB"
+	(label "5V"
 		(at 181.61 185.42 0)
 		(effects
@@
 		)
 	)
-	(label "5V"
-		(at 405.13 35.56 0)
-		(effects
-			(font
-				(size 1.27 1.27)
-			)
-			(justify left bottom)
-		)
-	)
 	(label "GND"
 		(at 125.73 166.37 180)
@@
 		)
 	)
-	(label "VUSB"
+	(label "5V"
 		(at 245.11 73.66 0)
 		(effects
@@
 		)
 	)
-	(label "VUSB"
-		(at 441.96 35.56 0)
-		(effects
-			(font
-				(size 1.27 1.27)
-			)
-			(justify left bottom)
-		)
-	)
 	(label "GND"
 		(at 125.73 184.15 180)
@@
 					(unit 1)
 				)
-			)
-		)
-	)
-	(symbol
-		(lib_id "Diode:MBR1020VL")
-		(at 420.37 35.56 180)
-		(unit 1)
-		(exclude_from_sim no)
-		(in_bom yes)
-		(on_board yes)
-		(dnp no)
-		(fields_autoplaced yes)
-		(property "Reference" "D5"
-			(at 420.6875 29.21 0)
-			(effects
-				(font
-					(size 1.27 1.27)
-				)
-			)
-		)
-		(property "Value" "MBR120VLSFT1G"
-			(at 420.6875 31.75 0)
-			(effects
-				(font
-					(size 1.27 1.27)
-				)
-			)
-		)
-		(property "Footprint" "Diode_SMD:D_SOD-123F"
-			(at 420.37 31.115 0)
-			(effects
-				(font
-					(size 1.27 1.27)
-				)
-				(hide yes)
-			)
-		)
-		(property "Datasheet" "https://www.onsemi.com/pub/Collateral/MBR1020VL-D.PDF"
-			(at 420.37 35.56 0)
-			(effects
-				(font
-					(size 1.27 1.27)
-				)
-				(hide yes)
-			)
-		)
-		(property "Description" "20V, 1A, 340 mV, Schottky Diode Rectifier, SOD-123F"
-			(at 420.37 35.56 0)
-			(effects
-				(font
-					(size 1.27 1.27)
-				)
-				(hide yes)
-			)
-		)
-		(pin "1"
-		)
-		(pin "2"
-		)
-		(instances
-			(project ""
-				(path "/04179b3e-2b25-41d4-a9af-8911a5c82cad"
-					(reference "D5")
-					(unit 1)
-				)

Commit message: pmos vtx power switching initial
Parts:
- added Q2, Q3: DMP3056L, Package_TO_SOT_SMD:SOT-23, symbol Transistor_FET:DMP3099L
- added R2: 10K, Resistor_SMD:R_0201_0603Metric, symbol Device:R
- Q1: value DMN3042L -> BSS138-7-F
Connections:
- net 12V: now also R1.1, Q2.2 (S); no longer J6.1 (Pin_1)
- net 5V: now also Q3.2 (S); no longer J7.1 (Pin_1)
- net GND: now also J6.2 (Pin_2), J7.2 (Pin_2), R2.2; no longer R1.2
- net VTX_GND: no longer J6.2 (Pin_2), J7.2 (Pin_2), Q1.3 (D)
- net VTX_PWR: now also R2.1; no longer R1.1
- new net VTX_12V: J6.1 (Pin_1), Q2.3 (D)
- new net VTX_5V: J7.1 (Pin_1), Q3.3 (D)
- new net VTX_GATE: Q1.3 (D), Q2.1 (G), Q3.1 (G), R1.2
Other:
- moved on the sheet: Q1, R1
