File: customboard/esc/esc.kicad_pcb (KiCad board)
At the start: 4 copper layers, 22.8 x 19 mm, 63 parts, among them J1 Conn_01x01_Pin, J10 Conn_01x03_Pin, J2 Conn_01x01_Pin, J3 Conn_01x01_Pin, J4 Conn_01x01_Pin, J5 Conn_01x01_Pin, J6 Conn_01x01_Pin, Q1 SQS140ELNW-T1_GE3, Q2 SQS140ELNW-T1_GE3, Q3 SQS140ELNW-T1_GE3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

Commit message: esc 4x
Parts:
- added J7: Conn_01x06, Connector_PinHeader_1.27mm:PinHeader_1x06_P1.27mm_Vertical, F.Cu at (170.4, 146.7)
- R10, R11, R4, R5, R7, R8: moved to F.Cu
- moved R9 57.5 mm to (169.6, 157.5)
- moved R6 57.5 mm to (169.6, 156.8)
- moved R10 54.6 mm to (169.6, 153.9), turned to 90 degrees
- moved R7 54.4 mm to (169.6, 155.8), turned to -90 degrees
- moved R3 53.6 mm to (168.6, 157.3), turned to -90 degrees
- moved R4 51.4 mm to (167.5, 157.6)
- moved U2 51.0 mm to (166.1, 147.8), turned to 180 degrees
- moved U1 49.5 mm to (166.1, 153.8), turned to 90 degrees
- moved R11 48.7 mm to (162.8, 145.1)
- moved C15 48.7 mm to (168.7, 150.4), turned to 90 degrees
- moved C24 46.1 mm to (163.1, 146.1), turned to -90 degrees
- moved R8 45.4 mm to (162.4, 146.7), turned to -90 degrees
- moved C22 44.7 mm to (163.5, 150.1), turned to -90 degrees
- moved R5 44.3 mm to (162.8, 150.5), turned to 90 degrees
- moved C23 43.9 mm to (162.6, 148.1), turned to -90 degrees
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Routing:
- net /BEMFC: track 12.6 -> 30.2 mm, vias 1 -> 3
- net /BEMFB: track 13.8 -> 29.4 mm, vias 1 -> 3
- net /BEMFA: track 11.2 -> 22.4 mm, vias 1 -> 3
- net /MOTORB: track 14.9 -> 25.3 mm, vias 1 -> 2
- net /MOTORC: track 21.5 -> 30.2 mm, vias 1 -> 2
- net /CLOW: track 7.39 -> 14.5 mm
- net /GHB: track 8.73 -> 15.8 mm, vias 1 -> 2
- net /GHC: track 12.6 -> 18.6 mm, vias 1 -> 2
- net /BLOW: track 6.09 -> 11.9 mm
- net /MOTORA: track 17.0 -> 22.3 mm, vias 1 -> 2
- net /ALOW: track 4.64 -> 9.20 mm
- net /BEMF_COMMON: track 5.76 -> 8.43 mm
- net /VOLTSENSE: track 8.28 -> 5.63 mm
- net /BOOSTA: track 2.99 -> 5.30 mm
- net +3.3V: track 0.32 -> 2.24 mm, vias 5 -> 6
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