File: customboard/esc/logic_board/single_esc.kicad_sch (KiCad schematic)
At the start: 26 parts, among them U1 STM32F051K8Ux, U2 DRV8300DRGE

Commit message: power board done, minor fixes in logic board
Parts:
- TP1, TP3: footprint TestPoint:TestPoint_Pad_D1.0mm -> Custom:SW_Testpoint
Changed lines of the file:
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@@
 			)
 		)
-		(property "Footprint" "TestPoint:TestPoint_Pad_D1.0mm"
+		(property "Footprint" "Custom:SW_Testpoint"
 			(at 213.36 114.3 0)
 			(effects
@@
 			)
 		)
-		(property "Footprint" "TestPoint:TestPoint_Pad_D1.0mm"
+		(property "Footprint" "Custom:SW_Testpoint"
 			(at 213.36 119.38 0)
 			(effects

Commit message: logic board 3v3 split
Connections:
- net +3.3V renamed 3V3
Changed lines of the file:
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@@
+		)
+	)
+	(hierarchical_label "3V3"
+		(shape input)
+		(at 53.34 19.05 90)
+		(effects
+			(font
+				(size 1.27 1.27)
+			)
+			(justify left)
 		)
 	)
@@
 					(unit 1)
 				)
-			)
-		)
-	)
-	(symbol
-		(lib_id "power:+3.3V")
-		(at 67.31 19.05 0)
-		(unit 1)
-		(exclude_from_sim no)
-		(in_bom yes)
-		(on_board yes)
-		(dnp no)
-		(fields_autoplaced yes)
-		(property "Reference" "#PWR020"
-			(at 67.31 22.86 0)
-			(effects
-				(font
-					(size 1.27 1.27)
-				)
-				(hide yes)
-			)
-		)
-		(property "Value" "+3.3V"
-			(at 67.31 13.97 0)
-			(effects
-				(font
-					(size 1.27 1.27)
-				)
-			)
-		)
-		(property "Footprint" ""
-			(at 67.31 19.05 0)
-			(effects
-				(font
-					(size 1.27 1.27)
-				)
-				(hide yes)
-			)
-		)
-		(property "Datasheet" ""
-			(at 67.31 19.05 0)
-			(effects
-				(font
-					(size 1.27 1.27)
-				)
-				(hide yes)
-			)
-		)
-		(property "Description" "Power symbol creates a global label with name \"+3.3V\""
-			(at 67.31 19.05 0)
-			(effects
-				(font
-					(size 1.27 1.27)
-				)
-				(hide yes)
-			)
-		)
-		(pin "1"
-		)
-		(instances
-			(project "logic_board"
-				(path "/42312c29-ac8b-461a-b58b-ac49287ed3f3/13cb8608-bedf-491a-b1ec-2ab011b3202c"
-					(reference "#PWR010")
-					(unit 1)
-				)
-				(path "/42312c29-ac8b-461a-b58b-ac49287ed3f3/97a9a163-8eb6-44fd-b320-4d1b4f4a0da0"
-					(reference "#PWR020")
-					(unit 1)
-				)
-				(path "/42312c29-ac8b-461a-b58b-ac49287ed3f3/ceb631f1-0d08-4424-a6aa-ea080f729a80"
-					(reference "#PWR039")
-					(unit 1)
-				)
-				(path "/42312c29-ac8b-461a-b58b-ac49287ed3f3/dceceb5a-1956-4d1e-895c-9f53784be5f2"
-					(reference "#PWR055")
-					(unit 1)
-				)

Commit message: narrower castelations on logic board; proper stls
Parts:
- C14, C15, C17, C21: value 100n -> 100n 10V
- C16, C20: value 10u -> 10u 10V
- C18, C22, C23, C24: value 1u -> 1u 10V
- C19: value 10n -> 10n 16V
- TP1, TP3: now left out of the parts list
Changed lines of the file:
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@@
 			)
 		)
-		(property "Value" "10n"
+		(property "Value" "10n 16V"
 			(at 104.14 25.3999 0)
 			(effects
@@
 			)
 		)
-		(property "Value" "1u"
+		(property "Value" "1u 10V"
 			(at 232.41 25.3999 0)
 			(effects
@@
 			)
 		)
-		(property "Value" "100n"
+		(property "Value" "100n 10V"
 			(at 167.64 25.3999 0)
 			(effects
@@
 			)
 		)
-		(property "Value" "10u"
+		(property "Value" "10u 10V"
 			(at 57.15 24.1299 0)
 			(effects
@@
 			)
 		)
-		(property "Value" "1u"
+		(property "Value" "1u 10V"
 			(at 86.36 25.3999 0)
 			(effects
@@
 			)
 		)
-		(property "Value" "100n"
+		(property "Value" "100n 10V"
 			(at 48.26 34.29 90)
 			(effects
@@
 			)
 		)
-		(property "Value" "10u"
+		(property "Value" "10u 10V"
 			(at 152.4 25.3999 0)
 			(effects
@@
 			)
 		)
-		(property "Value" "1u"
+		(property "Value" "1u 10V"
 			(at 232.41 38.0999 0)
 			(effects
@@
 			)
 		)
-		(property "Value" "1u"
+		(property "Value" "1u 10V"
 			(at 232.41 50.7999 0)
 			(effects
@@
 		(unit 1)
 		(exclude_from_sim no)
-		(in_bom yes)
+		(in_bom no)
 		(on_board yes)
 		(dnp no)
@@
 		(on_board yes)
 		(dnp no)
-		(fields_autoplaced yes)
 		(property "Reference" "C14"
 			(at 43.18 21.5899 0)
@@
 			)
 		)
-		(property "Value" "100n"
-			(at 43.18 24.1299 0)
+		(property "Value" "100n 10V"
+			(at 41.656 24.892 0)
 			(effects
 				(font
@@
 		(unit 1)
 		(exclude_from_sim no)
-		(in_bom yes)
+		(in_bom no)
 		(on_board yes)
 		(dnp no)
@@
 		(on_board yes)
 		(dnp no)
-		(fields_autoplaced yes)
 		(property "Reference" "C15"
 			(at 30.48 21.5899 0)
@@
 			)
 		)
-		(property "Value" "100n"
-			(at 30.48 24.1299 0)
-			(effects
-				(font
+		(property "Value" "100n 10V"
+			(at 28.448 24.892 0)
+			(effects
+				(font
