File: hardware/fc/droneboardh743_bga/droneboard.kicad_pcb (KiCad board)
At the start: 4 copper layers, 38 x 38 mm, 67 parts, among them J1 Conn_01x04_MountingPin, J10 Conn_01x03_Pin, J2 Conn_01x04_MountingPin, J3 Conn_01x08_MountingPin, J4 Conn_01x08_MountingPin, J5 USB_C_Receptacle_USB2.0_16P, J6 Conn_01x06_MountingPin, J7 Conn_01x06_MountingPin, Q1 DMN3042L, SW1 434133025816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

Commit message: high side pmos VTX switch
Parts:
- removed J7: Conn_01x06_MountingPin, Connector_JST:JST_SH_SM06B-SRSS-TB_1x06-1MP_P1.00mm_Horizontal
- removed R1: 10K, Resistor_SMD:R_0201_0603Metric
- added D5: YELLOW_LED, LED_SMD:LED_0603_1608Metric, F.Cu at (77.1, 110.6)
- added D6: YELLOW_LED, LED_SMD:LED_0603_1608Metric, F.Cu at (77.9, 108.8)
- added Q2: AO3401A, Package_TO_SOT_SMD:SOT-23, F.Cu at (78.5, 113.2)
- added Q3: 2SK3019, Package_TO_SOT_SMD:SOT-523, F.Cu at (74.2, 113.7)
- added Q4: AO3401A, Package_TO_SOT_SMD:SOT-23, F.Cu at (71.7, 115.8)
- added R12: 10K, Resistor_SMD:R_0201_0603Metric, F.Cu at (78.9, 117.6)
- added R15: 10K, Resistor_SMD:R_0201_0603Metric, F.Cu at (74.8, 111.8)
- added R16: 10K, Resistor_SMD:R_0201_0603Metric, F.Cu at (71.7, 114.2)
- added R17: 1K, Resistor_SMD:R_0402_1005Metric, F.Cu at (80.3, 109.9)
- added R2: 10K, Resistor_SMD:R_0201_0603Metric, F.Cu at (80.1, 113.2)
- J6: moved to B.Cu
- Q1: value DMN3042L -> 2SK3019; footprint Package_TO_SOT_SMD:SOT-23 -> Package_TO_SOT_SMD:SOT-523; moved to F.Cu
- moved Q1 5.59 mm to (79.1, 116.1), turned to 90 degrees
- turned J6 to 180 degrees
Connections:
- J6 pad 1: /12V -> /VTX_VCC
- J6 pad 2: /VTX_GND -> /GND
- Q1 pad 1: /VTX_PWR -> /VTX_PWR_5V
- Q1 pad 3: /VTX_GND -> Net-(Q1-D)
- U2 pad J9: /GND -> /VTX_PWR_5V
- U2 pad K9: /VTX_PWR -> /VTX_PWR_12V
Routing:
- net /VTX_PWR_5V: track 0.00 -> 13.7 mm
- net /VTX_PWR_12V: track 0.00 -> 7.46 mm
- net /VTX_PWR: track 5.99 -> 0.00 mm, vias 1 -> 0
- net /GND: track 56.4 -> 50.8 mm, vias 105 -> 107
- net /VTX_GND: track 5.48 -> 0.00 mm, vias 4 -> 0
- net /U7RX: track 14.7 -> 10.1 mm, vias 2 -> 1
- net Net-(D5-K): track 0.00 -> 3.72 mm
- net Net-(Q3-D): track 0.00 -> 2.89 mm
- net /U7TX: track 12.7 -> 10.0 mm, vias 2 -> 1
- net Net-(Q1-D): track 0.00 -> 2.52 mm
- net /RESET1: track 18.6 -> 20.5 mm
- net /12V: track 0.02 -> 1.51 mm, vias 10 -> 15
- net /5V: track 43.2 -> 44.7 mm, vias 30 -> 34
- net /VTX_VCC: vias 0 -> 9
- added copper zone on B.Cu, net /VTX_VCC
- added copper zone on F.Cu, net /VTX_VCC
- removed copper zone on B.Cu, net /VTX_GND
- removed copper zone on F.Cu, net /VTX_GND
