File: hardware/fc/droneboardh743_bga/droneboard.kicad_pcb (KiCad board)
At the start: 4 copper layers, 38 x 38 mm, 67 parts, among them J1 Conn_01x04_MountingPin, J10 Conn_01x03_Pin, J2 Conn_01x04_MountingPin, J3 Conn_01x08_MountingPin, J4 Conn_01x08_MountingPin, J5 USB_C_Receptacle_USB2.0_16P, J6 Conn_01x06_MountingPin, J7 Conn_01x06_MountingPin, Q1 DMN3042L, SW1 434133025816, SW2 434133025816, U1 TPS62933F, U2 STM32H743VIHx, U4 ICM-42688-P, U5 SPX3819M5-L-3-3, U6 SPX3819M5-L-3-3, Y2 CSTNE8M00G520000R0

Commit message: 9V regulator initial work
Parts:
- removed J3: Conn_01x08_MountingPin, Connector_JST:JST_SH_SM08B-SRSS-TB_1x08-1MP_P1.00mm_Horizontal
- removed J7: Conn_01x06_MountingPin, Connector_JST:JST_SH_SM06B-SRSS-TB_1x06-1MP_P1.00mm_Horizontal
- removed Q1: DMN3042L, Package_TO_SOT_SMD:SOT-23
- removed R1: 10K, Resistor_SMD:R_0201_0603Metric
- added C30: 10u50VX7R, Capacitor_SMD:C_1210_3225Metric, B.Cu at (66.7, 107.3)
- added C31: 10u50VX7R, Capacitor_SMD:C_1210_3225Metric, B.Cu at (61.4, 109.0)
- added C32: 100n50VX7R, Capacitor_SMD:C_0402_1005Metric, B.Cu at (62.8, 106.9)
- added C33: 33n50VX5R, Capacitor_SMD:C_0402_1005Metric, B.Cu at (64.1, 102.8)
- added C34: 100n50VX7R, Capacitor_SMD:C_0402_1005Metric, B.Cu at (63.1, 102.8)
- added C35: 22u10VX5R, Capacitor_SMD:C_0805_2012Metric, B.Cu at (56.8, 103.6)
- added C36: 22u10VX5R, Capacitor_SMD:C_0805_2012Metric, B.Cu at (54.9, 103.6)
- added C37: 100n, Capacitor_SMD:C_0201_0603Metric, B.Cu at (57.5, 101.2)
- added L2: XEL4030-332MEC, Inductor_SMD:L_Coilcraft_XxL4030, B.Cu at (60.1, 103.0)
- added R15: 5.49K, Resistor_SMD:R_0402_1005Metric, B.Cu at (65.5, 103.3)
- added R16: 1K, Resistor_SMD:R_0402_1005Metric, B.Cu at (66.0, 104.2)
- added U3: TPS62933F, Package_TO_SOT_SMD:SOT-583-8, B.Cu at (63.8, 105.1)
- H2, H4, H5, H6: footprint MountingHole:MountingHole_4.3mm_M4_DIN965 -> Custom:MountingHole_4.3mm_M4_Custom
- J4: moved to F.Cu
- J5: footprint Connector_USB:USB_C_Receptacle_GCT_USB4110 -> Custom:USB_C_Receptacle_GCT_USB4110_Custom
- U4: footprint footprints:LGA14_2P5X3X0P91_IVS-L -> Custom:LGA14_2P5X3X0P91_IVS-L_Custom
- moved C18 23.5 mm to (74.9, 116.7), turned to 90 degrees
- moved C27 22.6 mm to (72.3, 119.1), turned to 90 degrees
- moved C17 19.9 mm to (72.9, 116.7), turned to 90 degrees
- moved L1 16.5 mm to (69.7, 117.2), turned to 0 degrees
- moved C14 13.6 mm to (66.7, 117.4), turned to 90 degrees
- moved C29 13.0 mm to (65.7, 117.4), turned to 90 degrees
- moved R14 11.7 mm to (64.3, 117.0), turned to 180 degrees
- moved R13 9.83 mm to (63.8, 116.0), turned to 0 degrees
- moved U1 8.89 mm to (66.0, 115.2), turned to -90 degrees
- moved C20 8.28 mm to (68.3, 111.2), turned to 0 degrees
- moved C28 7.09 mm to (67.0, 113.3), turned to 180 degrees
- moved R7 3.41 mm to (69.8, 108.5), turned to 0 degrees
- moved R8 3.40 mm to (72.0, 109.2)
- moved C13 2.59 mm to (63.1, 112.9), turned to -90 degrees
- moved J4 0.09 mm to (63.5, 116.7), turned to 0 degrees
Connections:
- net /SMPS_BOOST renamed /SMPS_BOOST_9V
- net /SMPS_V renamed /SMPS_V_9V
- net /VFB renamed /VFB_9V
- C17 pad 1: /5V -> /9V
- C18 pad 1: /5V -> /9V
- C27 pad 2: /5V -> /9V
- J4 pad 3: /MOTOR3 -> /MOTOR0
- J4 pad 4: /MOTOR2 -> /MOTOR1
- J4 pad 5: /MOTOR0 -> /MOTOR3
- J4 pad 6: /MOTOR1 -> /MOTOR2
- J6 pad 1: /12V -> /9V
- J6 pad 2: /VTX_GND -> /GND
- J6 pad 3: /U7TX -> /U7RX
- J6 pad 4: /U7RX -> /U7TX
- L1 pad 2: /5V -> /9V
- R14 pad 2: /5V -> /9V
- U1 pad 2: unconnected-(U1-EN-Pad2) -> /VTX_PWR
Routing:
- net /VTX_PWR: track 5.99 -> 18.7 mm, vias 1 -> 2
- net /VTX_GND: track 5.48 -> 0.00 mm, vias 4 -> 0
- net /MOTOR1: track 22.2 -> 17.1 mm, vias 1 -> 0
- net /U7RX: track 14.7 -> 10.1 mm
- net /MOTOR2: track 22.7 -> 19.2 mm, vias 1 -> 0
- net /VBATMON: track 9.43 -> 6.15 mm
- net /U7TX: track 12.7 -> 10.0 mm
- net /SMPS_BOOST_5V: track 0.00 -> 1.23 mm
- net Net-(U3-SS): track 0.00 -> 1.07 mm
- net /9V: track 0.00 -> 1.05 mm, vias 0 -> 11
- net /MOTOR3: track 19.4 -> 18.4 mm, vias 1 -> 0
- net /MOTOR0: track 19.3 -> 18.8 mm, vias 1 -> 0
- net /5V: track 43.2 -> 43.5 mm, vias 30 -> 18
- net /12V: track 0.02 -> 0.00 mm, vias 10 -> 9
- net /GND: vias 105 -> 117
- added copper zone on B.Cu, net /9V
- added copper zone on F.Cu, net /9V
- added copper zone on In2.Cu, net /9V
- added copper zone on B.Cu, net /SMPS_V_5V
- removed copper zone on B.Cu, net /VTX_GND
- removed copper zone on F.Cu, net /VTX_GND

Commit message: stuff
Parts:
- J4: value Conn_01x08_MountingPin -> EscConnector8Pin
- J5: footprint Custom:USB_C_Receptacle_GCT_USB4110_Custom -> Connector_USB:USB_C_Receptacle_GCT_USB4110
- R14: value 5.49K -> 10.5K
- moved L1 0.16 mm to (69.5, 117.2)
- moved C23 0.16 mm to (71.5, 91.4)
- moved C22 0.15 mm to (76.3, 93.2)
Routing:
- net /GND: track 56.4 -> 2.31 mm, vias 117 -> 120
- net /5V: track 43.5 -> 23.2 mm, vias 18 -> 19
- net /VMCU: track 26.7 -> 22.9 mm
- net /9V: vias 11 -> 8
- added copper zone on F.Cu, net /VMCU
Other:
- board text added: "9"
