File: hardware/fc/droneboardh743_bga/droneboard.kicad_sch (KiCad schematic)
At the start: 67 parts, among them J1 Conn_01x04_MountingPin, J10 Conn_01x03_Pin, J2 Conn_01x04_MountingPin, J3 Conn_01x08_MountingPin, J4 Conn_01x08_MountingPin, J5 USB_C_Receptacle_USB2.0_16P, J6 Conn_01x06_MountingPin, J7 Conn_01x06_MountingPin, Q1 DMN3042L, SW1 434133025816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

Commit message: high side pmos VTX switch
Parts:
- removed J7: Conn_01x06_MountingPin, Connector_JST:JST_SH_SM06B-SRSS-TB_1x06-1MP_P1.00mm_Horizontal, symbol Connector_Generic_MountingPin:Conn_01x06_MountingPin
- removed Q1: DMN3042L, Package_TO_SOT_SMD:SOT-23, symbol Transistor_FET:DMN3042L
- removed R1: 10K, Resistor_SMD:R_0201_0603Metric, symbol Device:R
- added D5, D6: YELLOW_LED, LED_SMD:LED_0603_1608Metric, symbol Device:LED
- added Q1, Q3: 2SK3019, Package_TO_SOT_SMD:SOT-523, symbol Transistor_FET:2SK3019
- added Q2, Q4: AO3401A, Package_TO_SOT_SMD:SOT-23, symbol Transistor_FET:AO3401A
- added R12, R15, R16, R2: 10K, Resistor_SMD:R_0201_0603Metric, symbol Device:R
- added R17: 1K, Resistor_SMD:R_0402_1005Metric, symbol Device:R
Connections:
- net VTX_GND is gone; now on net GND: J6.2 (Pin_2)
- net 12V: now also Q4.2 (S), R16.2; no longer J6.1 (Pin_1)
- net 5V: now also Q2.2 (S), R2.2
- net GND: now also Q1.2 (S), Q3.2 (S), R12.2, R15.2, R17.2; no longer U2.J9 (PD9)
- net VTX_PWR renamed VTX_PWR_12V
- net VTX_PWR_12V: now also D6.2 (A), Q3.1 (G), R15.1
- new net: Q3.3 (D), Q4.1 (G), R16.1
- new net: D5.1 (K), D6.1 (K), R17.1
- new net: Q1.3 (D), Q2.1 (G), R2.1
- new net VTX_PWR_5V: D5.2 (A), Q1.1 (G), R12.1, U2.J9 (PD9)
- new net VTX_VCC: J6.1 (Pin_1), Q2.3 (D), Q4.3 (D)
- no-connect marks 14 -> 12
