File: hardware/fc/droneboardh743_bga/droneboard.kicad_sch (KiCad schematic)
At the start: 67 parts, among them J1 Conn_01x04_MountingPin, J10 Conn_01x03_Pin, J2 Conn_01x04_MountingPin, J3 Conn_01x08_MountingPin, J4 Conn_01x08_MountingPin, J5 USB_C_Receptacle_USB2.0_16P, J6 Conn_01x06_MountingPin, J7 Conn_01x06_MountingPin, Q1 DMN3042L, SW1 434133025816, SW2 434133025816, U1 TPS62933F, U2 STM32H743VIHx, U4 ICM-42688-P, U5 SPX3819M5-L-3-3, U6 SPX3819M5-L-3-3, Y2 CSTNE8M00G520000R0

Commit message: 9V regulator initial work
Parts:
- removed J3: Conn_01x08_MountingPin, Connector_JST:JST_SH_SM08B-SRSS-TB_1x08-1MP_P1.00mm_Horizontal, symbol Connector_Generic_MountingPin:Conn_01x08_MountingPin
- removed J7: Conn_01x06_MountingPin, Connector_JST:JST_SH_SM06B-SRSS-TB_1x06-1MP_P1.00mm_Horizontal, symbol Connector_Generic_MountingPin:Conn_01x06_MountingPin
- removed Q1: DMN3042L, Package_TO_SOT_SMD:SOT-23, symbol Transistor_FET:DMN3042L
- removed R1: 10K, Resistor_SMD:R_0201_0603Metric, symbol Device:R
- added C30, C31: 10u50VX7R, Capacitor_SMD:C_1210_3225Metric, symbol Device:C
- added C32, C34: 100n50VX7R, Capacitor_SMD:C_0402_1005Metric, symbol Device:C
- added C33: 33n50VX5R, Capacitor_SMD:C_0402_1005Metric, symbol Device:C
- added C35, C36: 22u10VX5R, Capacitor_SMD:C_0805_2012Metric, symbol Device:C
- added C37: 100n, Capacitor_SMD:C_0201_0603Metric, symbol Device:C
- added L2: XEL4030-332MEC, Inductor_SMD:L_Coilcraft_XxL4030, symbol Device:L
- added R15: 5.49K, Resistor_SMD:R_0402_1005Metric, symbol Device:R
- added R16: 1K, Resistor_SMD:R_0402_1005Metric, symbol Device:R
- added U3: TPS62933F, Package_TO_SOT_SMD:SOT-583-8, symbol Regulator_Switching:TPS62933F
- H2, H4, H5, H6: footprint MountingHole:MountingHole_4.3mm_M4_DIN965 -> Custom:MountingHole_4.3mm_M4_Custom
- J5: footprint Connector_USB:USB_C_Receptacle_GCT_USB4110 -> Custom:USB_C_Receptacle_GCT_USB4110_Custom
- U4: footprint footprints:LGA14_2P5X3X0P91_IVS-L -> Custom:LGA14_2P5X3X0P91_IVS-L_Custom
Connections:
- net VTX_GND is gone; now on net GND: J6.2 (Pin_2)
- net 12V: now also C30.1, C31.1, C32.2, U3.3 (VIN); no longer J6.1 (Pin_1)
- net 5V: now also C35.1, C36.1, C37.2, L2.2, R15.2; no longer C17.1, C18.1, C27.2, L1.2, R14.2
- net GND: now also C30.2, C31.2, C32.1, C33.1, C35.2, C36.2, C37.1, R16.1, U3.1 (RT), U3.4 (GND)
- net MOTOR0: now also J4.3 (Pin_3); no longer J4.5 (Pin_5)
- net MOTOR1: now also J4.4 (Pin_4); no longer J4.6 (Pin_6)
- net MOTOR2: now also J4.6 (Pin_6); no longer J4.4 (Pin_4)
- net MOTOR3: now also J4.5 (Pin_5); no longer J4.3 (Pin_3)
- net U7RX: now also J6.3 (Pin_3); no longer J6.4 (Pin_4)
- net U7TX: now also J6.4 (Pin_4); no longer J6.3 (Pin_3)
- net VTX_PWR: now also U1.2 (EN)
- net SMPS_BOOST renamed SMPS_BOOST_9V
- net SMPS_V renamed SMPS_V_9V
- net VFB renamed VFB_9V
- new net: C33.2, U3.7 (SS)
- new net 9V: C17.1, C18.1, C27.2, J6.1 (Pin_1), L1.2, R14.2
- new net SMPS_BOOST_5V: C34.2, U3.6 (BST)
- new net SMPS_V_5V: C34.1, L2.1, U3.5 (SW)
- new net VFB_5V: R15.1, R16.2, U3.8 (FB)
- no-connect marks 14 -> 10

Commit message: stuff
Parts:
- J4: value Conn_01x08_MountingPin -> EscConnector8Pin; symbol Connector_Generic_MountingPin:Conn_01x08_MountingPin -> Custom:EscConnector8Pin
- J5: footprint Custom:USB_C_Receptacle_GCT_USB4110_Custom -> Connector_USB:USB_C_Receptacle_GCT_USB4110
- R14: value 5.49K -> 10.5K
Connections:
- net GND: now also J5.SH (SHIELD); no longer J5.S1 (SHIELD)
Other:
- moved on the sheet: C1, C13, C14, C17, C18, C19, C2, C20, C21, C22, C23, C24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
